File: pcb/AirQMon.kicad_pcb (KiCad board)
At the start: 2 copper layers, 65 x 56 mm, 26 parts, among them J1 RaspberryPi Header, J2 NOX_PRE, J3 ADC Header, U1 BME280, U2 TGS2600, U3 RTC_hat, U4 MiCS-4514_BREAKOUT, U5 GPS_Breakout, U6 MCP3008

Commit message: Silk screen cleanup
Parts:
- added C1: 0.1u, Capacitors_THT:C_Disc_D3.8mm_W2.6mm_P2.50mm, F.Cu at (73.7, 83.3)
- added C2: 10u, Capacitors_THT:CP_Radial_D5.0mm_P2.00mm, F.Cu at (62.2, 95.2)
- added J4: ADC1, Pin_Headers:Pin_Header_Straight_1x01_Pitch2.54mm, F.Cu at (77.5, 101.6)
- added J5: ADC4, Pin_Headers:Pin_Header_Straight_1x01_Pitch2.54mm, F.Cu at (81.3, 101.6)
- U4: value MiCS-4514_BREAKOUT -> MiCS-4514
- U5: value GPS_Breakout -> GPS Breakout
- moved J3 9.52 mm to (53.3, 87.6)
- moved U5 8.89 mm to (53.3, 71.1), turned to 180 degrees
- moved U3 3.59 mm to (61.0, 61.0)
Connections:
- J1 pad 17: +3V3 -> (no net)
- MK1 pad 1: GND -> (no net)
- MK2 pad 1: GND -> (no net)
- MK3 pad 1: GND -> (no net)
- MK4 pad 1: GND -> (no net)
- U6 pad 1: (no net) -> Net-(J4-Pad1)
- U6 pad 5: (no net) -> Net-(J5-Pad1)
Routing:
- net +3V3: track 0.00 -> 149.2 mm, vias 0 -> 1
- net +5V: track 0.00 -> 139.0 mm, vias 0 -> 1
- net TGS_OUT: track 0.00 -> 55.1 mm, vias 0 -> 2
- net Net-(J3-Pad8): track 0.00 -> 53.9 mm
- net SDA: track 0.00 -> 52.1 mm, vias 0 -> 4
- net SCL: track 0.00 -> 49.8 mm, vias 0 -> 4
- net Net-(J3-Pad6): track 0.00 -> 42.2 mm
- net CS_ADC: track 0.00 -> 39.0 mm, vias 0 -> 2
- net MOSI: track 0.00 -> 38.8 mm, vias 0 -> 3
- net SCLK: track 0.00 -> 37.3 mm, vias 0 -> 2
- net MISO: track 0.00 -> 36.2 mm, vias 0 -> 2
- net Net-(J3-Pad4): track 0.00 -> 30.7 mm
- net ADC6: track 0.00 -> 27.8 mm, vias 0 -> 1
- net TXD: track 0.00 -> 26.7 mm, vias 0 -> 1
- net RXD: track 0.00 -> 26.1 mm
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- added copper zone on B.Cu, net GND
- added copper zone on F.Cu, net GND
Other:
- outline, holes or cut-outs redrawn
- board text added: "3V3 A6 A7 A8"
- board text added: "5V| GND| GND| GND|"
- board text added: "AirQMon Env Sensr v0.1"
- board text added: "VCC"
- board text added: "https://github.com/PhirePhly/AirQMon"
